Commit message: updated

File: src/mobile_robot/description/robot_core.xacro (robot description, xacro)
@@ -53,5 +53,5 @@
     </link>
     <gazebo reference="chassis">
-        <material>Gazebo/White</material>
+        <material>Gazebo/Yellow</material>
     </gazebo>
     <!-- LEFT WHEEL LINK -->
